Commit message: it all works!

File: descriptions/panda/panda.urdf (robot description, URDF)
Before this commit: robot panda, 13 links, 12 joints
Links:
- link panda_hand: geometry collision mesh filename=package://meshes/collision/hand.obj
- link panda_link8: geometry visual mesh filename=package://meshes/visual/link8.obj
